Commit message: update：1.选择优化arm逆运动学求解器   2.增加自体碰撞检测密度   3.降低仿真底盘速度

File: whole_description/urdf/multi_robot.urdf.xacro (robot description, xacro)
@@ -10,6 +10,6 @@
         <child link="chassis_x_link"/>
         <axis xyz="1 0 0"/> <!-- 沿 X 轴 -->
-        <limit lower="-1.0" upper="1.0" effort="100.0" velocity="10.0"/> <!-- 根据需要调整范围 -->
-        <origin xyz="0.34 0.51 0" rpy="0 0 3.1415"/>
+        <limit lower="-1.0" upper="1.0" effort="50.0" velocity="5.0"/> <!-- 根据需要调整范围 -->
+        <origin xyz="0.38 0.47 0" rpy="0 0 3.1415"/>
     </joint>
     <link
@@ -26,5 +26,5 @@
         <child link="chassis_y_link"/>
         <axis xyz="0 1 0"/> <!-- 沿 Y 轴 -->
-        <limit lower="-1.0" upper="1.0" effort="100.0" velocity="10.0"/> <!-- 根据需要调整范围 -->
+        <limit lower="-1.0" upper="1.0" effort="50.0" velocity="5.0"/> <!-- 根据需要调整范围 -->
         <origin xyz="0 0 0" rpy="0 0 0"/>
     </joint>
@@ -42,5 +42,5 @@
         <child link="footprint_link"/>
         <axis xyz="0 0 1"/> <!-- 绕 Z 轴 -->
-        <limit lower="-3.1415" upper="3.1415" effort="100.0" velocity="10.0"/> <!-- 根据需要调整范围 -->
+        <limit lower="-3.1415" upper="3.1415" effort="50.0" velocity="5.0"/> <!-- 根据需要调整范围 -->
         <origin xyz="0 0 0" rpy="0 0 0"/>
     </joint>

Commit message: update：1.添加spin node  2.添加底盘运动逻辑，未实现成功执行

File: whole_description/urdf/multi_robot.urdf.xacro (robot description, xacro)
@@ -10,5 +10,5 @@
         <child link="chassis_x_link"/>
         <axis xyz="1 0 0"/> <!-- 沿 X 轴 -->
-        <limit lower="-1.0" upper="1.0" effort="50.0" velocity="5.0"/> <!-- 根据需要调整范围 -->
+        <limit lower="-1.0" upper="1.0" effort="100.0" velocity="10.0"/> <!-- 根据需要调整范围 -->
         <origin xyz="0.38 0.47 0" rpy="0 0 3.1415"/>
     </joint>
@@ -26,5 +26,5 @@
         <child link="chassis_y_link"/>
         <axis xyz="0 1 0"/> <!-- 沿 Y 轴 -->
-        <limit lower="-1.0" upper="1.0" effort="50.0" velocity="5.0"/> <!-- 根据需要调整范围 -->
+        <limit lower="-1.0" upper="1.0" effort="100.0" velocity="10.0"/> <!-- 根据需要调整范围 -->
         <origin xyz="0 0 0" rpy="0 0 0"/>
     </joint>
@@ -42,5 +42,5 @@
         <child link="footprint_link"/>
         <axis xyz="0 0 1"/> <!-- 绕 Z 轴 -->
-        <limit lower="-3.1415" upper="3.1415" effort="50.0" velocity="5.0"/> <!-- 根据需要调整范围 -->
+        <limit lower="-3.1415" upper="3.1415" effort="100.0" velocity="10.0"/> <!-- 根据需要调整范围 -->
         <origin xyz="0 0 0" rpy="0 0 0"/>
     </joint>
