Commit message: update：1.取消chassis_group，把底盘添加到arm_group里面    2.机械改长link6

File: engineer_description/urdf/engineer_total.urdf.xacro (robot description, xacro)
@@ -339,8 +339,8 @@
   <joint
     name="J0_joint"
-    type="continuous">
+    type="revolute">
     <origin
       xyz="0.057679 0.0009078 0.136"
-      rpy="0 0 0.802825" />
+      rpy="0 0 0.102825" />
     <parent
       link="base_Link" />
@@ -349,4 +349,9 @@
     <axis
       xyz="0 0 1" />
+    <limit
+      lower="-3.14"
+      upper="3.14"
+      effort="100"
+      velocity="100" />
   </joint>
   <link
@@ -635,6 +640,6 @@
       xyz="0 0 1" />
     <limit
-      lower="1.74"
-      upper="4.54"
+      lower="1.31"
+      upper="4.97"
       effort="60"
       velocity="5" />
@@ -644,15 +649,15 @@
     <inertial>
       <origin
-        xyz="2.3269E-11 3.2741E-11 0.14165"
-        rpy="0 0 0" />
-      <mass
-        value="7.7518" />
-      <inertia
-        ixx="0.048485"
-        ixy="1.4848E-08"
-        ixz="2.045E-11"
-        iyy="0.048485"
-        iyz="5.3943E-12"
-        izz="0.048493" />
+        xyz="-1.23475841270343E-09 4.03415967298315E-09 0.0278757307831412"
+        rpy="0 0 0" />
+      <mass
+        value="0.178143267563857" />
+      <inertia
+        ixx="0.000129094390101851"
+        ixy="1.48506907428467E-08"
+        ixz="2.40814672934691E-11"
+        iyy="0.000129030586750178"
+        iyz="2.41689552037147E-11"
+        izz="7.00687059355998E-05" />
     </inertial>
     <visual>
@@ -667,5 +672,5 @@
         name="">
         <color
-          rgba="0.89804 0.91765 0.92941 1" />
+          rgba="0.898039215686275 0.917647058823529 0.929411764705882 1" />
       </material>
     </visual>
@@ -684,6 +689,6 @@
     type="revolute">
     <origin
-      xyz="-0.00016514 0.0037607 0.048001"
-      rpy="1.5962 -1.5708 0" />
+      xyz="-0.000514233258821717 0.00374244231316156 0.0480008261045562"
+      rpy="1.64994041161029 -1.5707963267949 0" />
     <parent
       link="J5" />
@@ -700,9 +705,41 @@
   <link
     name="mine_link">
-    <visual>
-      <origin
-        xyz="0 0 0"
-        rpy="0 0 0" />
-    </visual>
+    <inertial>
+      <origin
+        xyz="0.00259034918237153 0.000383105433044262 0.102689008639284"
+        rpy="0 0 0" />
+      <mass
+        value="7.49632983624276" />
+      <inertia
+        ixx="0.0469714949950914"
+        ixy="1.85907797157586E-07"
+        ixz="2.41999667470607E-05"
+        iyy="0.0468593512484876"
+        iyz="4.01177085607054E-08"
+        izz="0.0469679528165848" />
+    </inertial>
+    <visual>
+      <origin
+        xyz="0 0 0"
+        rpy="0 0 0" />
+      <geometry>
+        <mesh
+          filename="package://engineer_description/meshes/end.STL" />
+      </geometry>
+      <material
+        name="">
+        <color
+          rgba="0.298039215686275 0.298039215686275 0.298039215686275 1" />
+      </material>
+    </visual>
+    <collision>
+      <origin
+        xyz="0 0 0"
+        rpy="0 0 0" />
+      <geometry>
+        <mesh
+          filename="package://engineer_description/meshes/end.STL" />
+      </geometry>
+    </collision>
   </link>
   <joint
@@ -710,10 +747,31 @@
     type="fixed">
     <origin
-      xyz="0 0 0.25"
+      xyz="0 0 0.0704957805907174"
+      rpy="0 0 0" />
+    <parent
+      link="J6" />
+    <child
+      link="mine_link" />
+    <axis
+      xyz="0 0 0" />
+  </joint>
+  <link
+    name="endface_link">
+    <visual>
+      <origin
+        xyz="0 0 0"
+        rpy="0 0 0" />
+    </visual>
+  </link>
+  <joint
+    name="endface_joint"
+    type="fixed">
+    <origin
+      xyz="0 0 0.20"
       rpy="-1.57 1.57 0" />
     <parent
-      link="J6" />
-    <child
       link="mine_link" />
+    <child
+      link="endface_link" />
     <axis
       xyz="0 0 0" />

File: whole_config/config/multi_robot.ros2_control.xacro (robot description, xacro)
@@ -57,8 +57,22 @@
                 <state_interface name="velocity"/>
             </joint>
-            <joint name="chassis">
+            <joint name="chassis_x">
                 <command_interface name="position"/>
                 <state_interface name="position">
-                  <param name="initial_value">${initial_positions['chassis']}</param>
+                  <param name="initial_value">${initial_positions['chassis_x']}</param>
+                </state_interface>
+                <state_interface name="velocity"/>
+            </joint>
+            <joint name="chassis_y">
+                <command_interface name="position"/>
+                <state_interface name="position">
+                  <param name="initial_value">${initial_positions['chassis_y']}</param>
+                </state_interface>
+                <state_interface name="velocity"/>
+            </joint>
+            <joint name="chassis_theta">
+                <command_interface name="position"/>
+                <state_interface name="position">
+                  <param name="initial_value">${initial_positions['chassis_theta']}</param>
                 </state_interface>
                 <state_interface name="velocity"/>

File: whole_description/urdf/multi_robot.urdf.xacro (robot description, xacro)
@@ -5,8 +5,43 @@
     <!-- 1. 载入第一个机器人 (带底盘机械臂) -->
     <xacro:include filename="$(find engineer_description)/urdf/engineer_total.urdf.xacro"/>
-    <joint name="chassis" type="planar">
+    <!-- 沿 X 轴的棱柱关节 -->
+    <joint name="chassis_x" type="prismatic">
         <parent link="root_link"/>
+        <child link="chassis_x_link"/>
+        <axis xyz="1 0 0"/> <!-- 沿 X 轴 -->
+        <limit lower="-1.0" upper="1.0" effort="100.0" velocity="10.0"/> <!-- 根据需要调整范围 -->
+        <origin xyz="0.34 0.51 0" rpy="0 0 3.1415"/>
+    </joint>
+    <link
+    name="chassis_x_link">
+    <visual>
+      <origin
+        xyz="0 0 0"
+        rpy="0 0 0" />
+    </visual>
+   </link>
+    <!-- 沿 Y 轴的棱柱关节 -->
+    <joint name="chassis_y" type="prismatic">
+        <parent link="chassis_x_link"/>
+        <child link="chassis_y_link"/>
+        <axis xyz="0 1 0"/> <!-- 沿 Y 轴 -->
+        <limit lower="-1.0" upper="1.0" effort="100.0" velocity="10.0"/> <!-- 根据需要调整范围 -->
+        <origin xyz="0 0 0" rpy="0 0 0"/>
+    </joint>
+    <link
+    name="chassis_y_link">
+    <visual>
+      <origin
+        xyz="0 0 0"
+        rpy="0 0 0" />
+    </visual>
+   </link>
+    <!-- 绕 Z 轴的旋转关节 -->
+    <joint name="chassis_theta" type="revolute">
+        <parent link="chassis_y_link"/>
         <child link="footprint_link"/>
-        <origin xyz="0.38 0.60 0" rpy="0 0 2.355"/>
+        <axis xyz="0 0 1"/> <!-- 绕 Z 轴 -->
+        <limit lower="-3.1415" upper="3.1415" effort="100.0" velocity="10.0"/> <!-- 根据需要调整范围 -->
+        <origin xyz="0 0 0" rpy="0 0 0"/>
     </joint>
     <!-- 2. 载入第二个机器人 (固定机械臂 + 箱子) -->

Commit message: update:机械臂改回原来长度，取消底盘旋转关节

File: engineer_description/urdf/engineer_total.urdf.xacro (robot description, xacro)
@@ -349,5 +349,5 @@
     <axis
       xyz="0 0 1" />
-    <limit
+<limit
       lower="-3.14"
       upper="3.14"
@@ -640,6 +640,6 @@
       xyz="0 0 1" />
     <limit
-      lower="1.31"
-      upper="4.97"
+      lower="1.74"
+      upper="4.54"
       effort="60"
       velocity="5" />
@@ -649,15 +649,15 @@
     <inertial>
       <origin
-        xyz="-1.23475841270343E-09 4.03415967298315E-09 0.0278757307831412"
-        rpy="0 0 0" />
-      <mass
-        value="0.178143267563857" />
-      <inertia
-        ixx="0.000129094390101851"
-        ixy="1.48506907428467E-08"
-        ixz="2.40814672934691E-11"
-        iyy="0.000129030586750178"
-        iyz="2.41689552037147E-11"
-        izz="7.00687059355998E-05" />
+        xyz="2.3269E-11 3.2741E-11 0.14165"
+        rpy="0 0 0" />
+      <mass
+        value="7.7518" />
+      <inertia
+        ixx="0.048485"
+        ixy="1.4848E-08"
+        ixz="2.045E-11"
+        iyy="0.048485"
+        iyz="5.3943E-12"
+        izz="0.048493" />
     </inertial>
     <visual>
@@ -672,5 +672,5 @@
         name="">
         <color
-          rgba="0.898039215686275 0.917647058823529 0.929411764705882 1" />
+          rgba="0.89804 0.91765 0.92941 1" />
       </material>
     </visual>
@@ -689,6 +689,6 @@
     type="revolute">
     <origin
-      xyz="-0.000514233258821717 0.00374244231316156 0.0480008261045562"
-      rpy="1.64994041161029 -1.5707963267949 0" />
+      xyz="-0.00016514 0.0037607 0.048001"
+      rpy="1.5962 -1.5708 0" />
     <parent
       link="J5" />
@@ -705,41 +705,9 @@
   <link
     name="mine_link">
-    <inertial>
-      <origin
-        xyz="0.00259034918237153 0.000383105433044262 0.102689008639284"
-        rpy="0 0 0" />
-      <mass
-        value="7.49632983624276" />
-      <inertia
-        ixx="0.0469714949950914"
-        ixy="1.85907797157586E-07"
-        ixz="2.41999667470607E-05"
-        iyy="0.0468593512484876"
-        iyz="4.01177085607054E-08"
-        izz="0.0469679528165848" />
-    </inertial>
-    <visual>
-      <origin
-        xyz="0 0 0"
-        rpy="0 0 0" />
-      <geometry>
-        <mesh
-          filename="package://engineer_description/meshes/end.STL" />
-      </geometry>
-      <material
-        name="">
-        <color
-          rgba="0.298039215686275 0.298039215686275 0.298039215686275 1" />
-      </material>
-    </visual>
-    <collision>
-      <origin
-        xyz="0 0 0"
-        rpy="0 0 0" />
-      <geometry>
-        <mesh
-          filename="package://engineer_description/meshes/end.STL" />
-      </geometry>
-    </collision>
+    <visual>
+      <origin
+        xyz="0 0 0"
+        rpy="0 0 0" />
+    </visual>
   </link>
   <joint
@@ -747,6 +715,6 @@
     type="fixed">
     <origin
-      xyz="0 0 0.0704957805907174"
-      rpy="0 0 0" />
+      xyz="0 0 0.25"
+      rpy="-1.57 1.57 0" />
     <parent
       link="J6" />
@@ -756,24 +724,3 @@
       xyz="0 0 0" />
   </joint>
-  <link
-    name="endface_link">
-    <visual>
-      <origin
-        xyz="0 0 0"
-        rpy="0 0 0" />
-    </visual>
-  </link>
-  <joint
-    name="endface_joint"
-    type="fixed">
-    <origin
-      xyz="0 0 0.20"
-      rpy="-1.57 1.57 0" />
-    <parent
-      link="mine_link" />
-    <child
-      link="endface_link" />
-    <axis
-      xyz="0 0 0" />
-  </joint>
 </robot>

File: whole_config/config/multi_robot.ros2_control.xacro (robot description, xacro)
@@ -71,11 +71,4 @@
                 <state_interface name="velocity"/>
             </joint>
-            <joint name="chassis_theta">
-                <command_interface name="position"/>
-                <state_interface name="position">
-                  <param name="initial_value">${initial_positions['chassis_theta']}</param>
-                </state_interface>
-                <state_interface name="velocity"/>
-            </joint>
             <joint name="j0">
                 <command_interface name="position"/>

File: whole_description/urdf/multi_robot.urdf.xacro (robot description, xacro)
@@ -8,5 +8,5 @@
     <joint name="chassis_x" type="prismatic">
         <parent link="root_link"/>
-        <child link="chassis_x_link"/>
+        <child link="chassis_link"/>
         <axis xyz="1 0 0"/> <!-- 沿 X 轴 -->
         <limit lower="-1.0" upper="1.0" effort="100.0" velocity="10.0"/> <!-- 根据需要调整范围 -->
@@ -14,5 +14,5 @@
     </joint>
     <link
-    name="chassis_x_link">
+    name="chassis_link">
     <visual>
       <origin
@@ -23,24 +23,8 @@
     <!-- 沿 Y 轴的棱柱关节 -->
     <joint name="chassis_y" type="prismatic">
-        <parent link="chassis_x_link"/>
-        <child link="chassis_y_link"/>
+        <parent link="chassis_link"/>
+        <child link="footprint_link"/>
         <axis xyz="0 1 0"/> <!-- 沿 Y 轴 -->
-        <limit lower="-1.0" upper="1.0" effort="100.0" velocity="10.0"/> <!-- 根据需要调整范围 -->
-        <origin xyz="0 0 0" rpy="0 0 0"/>
-    </joint>
-    <link
-    name="chassis_y_link">
-    <visual>
-      <origin
-        xyz="0 0 0"
-        rpy="0 0 0" />
-    </visual>
-   </link>
-    <!-- 绕 Z 轴的旋转关节 -->
-    <joint name="chassis_theta" type="revolute">
-        <parent link="chassis_y_link"/>
-        <child link="footprint_link"/>
-        <axis xyz="0 0 1"/> <!-- 绕 Z 轴 -->
-        <limit lower="-3.1415" upper="3.1415" effort="100.0" velocity="10.0"/> <!-- 根据需要调整范围 -->
+        <limit lower="-1.5" upper="1.5" effort="100.0" velocity="10.0"/> <!-- 根据需要调整范围 -->
         <origin xyz="0 0 0" rpy="0 0 0"/>
     </joint>
